File: STM32G4xx_Cell_DevBoard.kicad_sch (KiCad schematic)
At the start: 55 parts, among them J1 Conn_02x12_Odd_Even, J2 Conn_02x12_Odd_Even, J3 Conn_01x04, J4 USB_C_Receptacle_USB2.0_16P, J5 Conn_01x14, SW1 SW_Push, U1 STM32G474CETx, U2 ME6211C33M5, U3 TPS54302, Y1 25MHz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

Commit message: 添加库文件并修改
Parts:
- R7: value 100k -> 75k
- R8: value 13.3k -> 10k
- SW1: footprint MyLibrary:3_4微动开关 -> Library:3_4微动开关
Changed lines of the file:
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@@
 			)
 		)
-		(property "Value" "100k"
+		(property "Value" "75k"
 			(at 227.33 68.58 90)
 			(effects
@@
 			)
 		)
-		(property "Footprint" "MyLibrary:3_4微动开关"
+		(property "Footprint" "Library:3_4微动开关"
 			(at 43.18 153.67 0)
 			(effects
@@
 			)
 		)
-		(property "Value" "13.3k"
+		(property "Value" "10k"
 			(at 218.44 81.2799 0)
 			(effects
